Commit message: ignore把rslrl干掉了

File: jump/resources/robots/infantry_V4/urdf/infantry_V4_increase.urdf (robot description, URDF)
Before this commit: robot infantry_V4, 7 links, 6 joints
Links:
- link base_link: geometry collision mesh filename=../../../../../plane/resources/robots/infantry_V4/meshes/ba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; visual mesh filename=../../../../../plane/resources/robots/infantry_V4/meshes/ba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
- link l_wheel_Link: geometry collision mesh filename=../../../../../plane/resources/robots/infantry_V4/meshes/l_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; visual mesh filename=../../../../../plane/resources/robots/infantry_V4/meshes/l_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
- link lf0_Link: geometry collision mesh filename=../../../../../plane/resources/robots/infantry_V4/meshes/lf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; visual mesh filename=../../../../../plane/resources/robots/infantry_V4/meshes/lf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
- link lf1_Link: geometry collision mesh filename=../../../../../plane/resources/robots/infantry_V4/meshes/lf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; visual mesh filename=../../../../../plane/resources/robots/infantry_V4/meshes/lf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
- link r_wheel_Link: geometry collision mesh filename=../../../../../plane/resources/robots/infantry_V4/meshes/r_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; visual mesh filename=../../../../../plane/resources/robots/infantry_V4/meshes/r_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
- link rf0_Link: geometry collision mesh filename=../../../../../plane/resources/robots/infantry_V4/meshes/rf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; visual mesh filename=../../../../../plane/resources/robots/infantry_V4/meshes/rf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
- link rf1_Link: geometry collision mesh filename=../../../../../plane/resources/robots/infantry_V4/meshes/rf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; visual mesh filename=../../../../../plane/resources/robots/infantry_V4/meshes/rf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
